Commit message: feat(gizmo_description): add multi-robot prefix support to urdf and display launch

File: src/gizmo_description/urdf/gizmo.urdf.xacro (robot description, xacro)
@@ -1,4 +1,8 @@
 <?xml version="1.0" ?>
 <robot name="gizmo" xmlns:xacro="http://www.ros.org/wiki/xacro">
+    <xacro:arg name="prefix" default="" />
+    <xacro:property name="_prefix" value="$(arg prefix)" />
+    <xacro:property name="tf_prefix" value="${_prefix if (_prefix == '' or _prefix.endswith('/')) else _prefix + '/'}" />
+    <xacro:property name="topic_prefix" value="${('/' + tf_prefix) if not tf_prefix.startswith('/') else tf_prefix}" />
     <xacro:include filename="$(find gizmo_description)/urdf/include/robot_components/gizmo_mobile_base.xacro" />
     <xacro:include filename="$(find gizmo_description)/urdf/include/gazebo_components/gizmo_mobile_base.gazebo.xacro" />

File: src/gizmo_description/urdf/include/gazebo_components/camera.gazebo.xacro (robot description, xacro)
@@ -5,15 +5,15 @@
     <xacro:property name="camera_type" value="$(arg camera_type)" />
     <!-- Camera Gazebo Plugin -->
-    <gazebo reference="camera_link">
+    <gazebo reference="${tf_prefix}camera_link">
         <sensor name="camera" type="${camera_type}">
             <pose>${camera_optical_frame_o_xyz} 0 0 0</pose>
             <xacro:if value="${camera_type == 'depth_camera'}">
-                <topic>camera/depth/image_raw</topic>
+                <topic>${topic_prefix}camera/depth/image_raw</topic>
             </xacro:if>
             <xacro:unless value="${camera_type == 'depth_camera'}">
-                <topic>camera/image_raw</topic>
+                <topic>${topic_prefix}camera/image_raw</topic>
             </xacro:unless>
-            <camera_info_topic>camera/camera_info</camera_info_topic>
-            <gz_frame_id>camera_optical_frame</gz_frame_id>
+            <camera_info_topic>${topic_prefix}camera/camera_info</camera_info_topic>
+            <gz_frame_id>${tf_prefix}camera_optical_frame</gz_frame_id>
             <update_rate>30</update_rate>
             <always_on>1</always_on>

File: src/gizmo_description/urdf/include/gazebo_components/gizmo_mobile_base.gazebo.xacro (robot description, xacro)
@@ -4,5 +4,5 @@
     <xacro:property name="wheel_radius" value="0.035" />
     <!-- Left Wheel Surface Friction & Contact Stability -->
-    <gazebo reference="wheel_left">
+    <gazebo reference="${tf_prefix}wheel_left">
         <mu1>1.0</mu1>
         <mu2>1.0</mu2>
@@ -14,5 +14,5 @@
     </gazebo>
     <!-- Right Wheel Surface Friction & Contact Stability -->
-    <gazebo reference="wheel_right">
+    <gazebo reference="${tf_prefix}wheel_right">
         <mu1>1.0</mu1>
         <mu2>1.0</mu2>
@@ -24,5 +24,5 @@
     </gazebo>
     <!-- Caster Wheel Surface Friction & Contact Stability (Sliding) -->
-    <gazebo reference="caster_wheel">
+    <gazebo reference="${tf_prefix}caster_wheel">
         <mu1>0.001</mu1>
         <mu2>0.001</mu2>
@@ -52,8 +52,8 @@
             <max_torque>5.0</max_torque>
             <!-- Topics & Frames -->
-            <topic>/cmd_vel</topic>
-            <odom_topic>/wheel_odom</odom_topic>
-            <frame_id>odom</frame_id>
-            <child_frame_id>base_footprint</child_frame_id>
+            <topic>${topic_prefix}cmd_vel</topic>
+            <odom_topic>${topic_prefix}wheel_odom</odom_topic>
+            <frame_id>${tf_prefix}odom</frame_id>
+            <child_frame_id>${tf_prefix}base_footprint</child_frame_id>
             <!-- Publishing Options -->
             <publish_odom>true</publish_odom>
@@ -63,5 +63,5 @@
         <!-- Joint State Publisher Plugin for Gazebo -->
         <plugin filename="gz-sim-joint-state-publisher-system" name="gz::sim::systems::JointStatePublisher">
-            <topic>/joint_states</topic>
+            <topic>${topic_prefix}joint_states</topic>
             <joint_name>left_wheel_joint</joint_name>
             <joint_name>right_wheel_joint</joint_name>

File: src/gizmo_description/urdf/include/gazebo_components/imu.gazebo.xacro (robot description, xacro)
@@ -2,10 +2,10 @@
 <robot xmlns:xacro="http://www.ros.org/wiki/xacro">
     <!-- Gazebo Plugin Configuration -->
-    <gazebo reference="imu_link">
+    <gazebo reference="${tf_prefix}imu_link">
         <sensor name="imu" type="imu">
             <always_on>true</always_on>
             <update_rate>100</update_rate>
-            <gz_frame_id>imu_link</gz_frame_id>
-            <topic>imu</topic>
+            <gz_frame_id>${tf_prefix}imu_link</gz_frame_id>
+            <topic>${topic_prefix}imu/data</topic>
             <imu>
                 <angular_velocity>

File: src/gizmo_description/urdf/include/gazebo_components/lidar.gazebo.xacro (robot description, xacro)
@@ -2,9 +2,9 @@
 <robot xmlns:xacro="http://www.ros.org/wiki/xacro">
     <!-- Gazebo Harmonic GPU 2D LiDAR Plugin (SDF 1.10 Specification) -->
-    <gazebo reference="scan_frame">
+    <gazebo reference="${tf_prefix}scan_frame">
         <sensor name="gpu_lidar" type="gpu_lidar">
-            <pose relative_to="scan_frame">0 0 0 0 0 0</pose>
-            <topic>scan</topic>
-            <frame_id>scan_frame</frame_id>
+            <pose relative_to="${tf_prefix}scan_frame">0 0 0 0 0 0</pose>
+            <topic>${topic_prefix}scan</topic>
+            <frame_id>${tf_prefix}scan_frame</frame_id>
             <update_rate>10</update_rate>
             <always_on>true</always_on>

File: src/gizmo_description/urdf/include/gazebo_components/sensors.gazebo.xacro (robot description, xacro)
@@ -1,10 +1,4 @@
 <?xml version="1.0" ?>
 <robot xmlns:xacro="http://www.ros.org/wiki/xacro">
-    <!-- sensor system plugin for gazebo -->
-    <gazebo>
-        <plugin name='gz::sim::systems::Sensors' filename='gz-sim-sensors-system'>
-            <render_engine>ogre2</render_engine>
-        </plugin>
-    </gazebo>
     <!-- Sensor toggles -->
     <xacro:arg name="use_lidar" default="true"/>

File: src/gizmo_description/urdf/include/robot_components/base_floor1.xacro (robot description, xacro)
@@ -7,5 +7,5 @@
     <xacro:property name="base_floor1_o_rpy" value="0 0 0" />
     <!-- Link base_floor1 -->
-    <link name="base_floor1">
+    <link name="${tf_prefix}base_floor1">
         <xacro:cylinder_inertia m="${base_floor1_m}" r="${base_floor1_r}" h="${base_floor1_h}" o_xyz="${base_floor1_o_xyz}" o_rpy="${base_floor1_o_rpy}"/>
         <collision>

File: src/gizmo_description/urdf/include/robot_components/base_floor2.xacro (robot description, xacro)
@@ -7,5 +7,5 @@
     <xacro:property name="base_floor2_o_rpy" value="0 0 0" />
     <!-- Link base_floor2 -->
-    <link name="base_floor2">
+    <link name="${tf_prefix}base_floor2">
         <xacro:cylinder_inertia m="${base_floor2_m}" r="${base_floor2_r}" h="${base_floor2_h}" o_xyz="${base_floor2_o_xyz}" o_rpy="${base_floor2_o_rpy}"/>
         <collision>

File: src/gizmo_description/urdf/include/robot_components/base_floor3.xacro (robot description, xacro)
@@ -7,5 +7,5 @@
     <xacro:property name="base_floor3_o_rpy" value="0 0 0" />
     <!-- Link base_floor3 -->
-    <link name="base_floor3">
+    <link name="${tf_prefix}base_floor3">
         <xacro:cylinder_inertia m="${base_floor3_m}" r="${base_floor3_r}" h="${base_floor3_h}" o_xyz="${base_floor3_o_xyz}" o_rpy="${base_floor3_o_rpy}"/>
         <collision>

File: src/gizmo_description/urdf/include/robot_components/camera.xacro (robot description, xacro)
@@ -9,5 +9,5 @@
     <xacro:property name="camera_o_rpy" value="0 0 0" />
   <!-- Link realsense_d435 -->
-  <link name="camera_link">
+  <link name="${tf_prefix}camera_link">
     <xacro:box_inertia m="${camera_m}" x="${camera_length}" y="${camera_width}" z="${camera_height}" o_xyz="${camera_o_xyz}" o_rpy="${camera_o_rpy}"/>
     <collision>
@@ -28,4 +28,4 @@
     </visual>
   </link>
-  <link name="camera_optical_frame"/>
+  <link name="${tf_prefix}camera_optical_frame"/>
 </robot>

File: src/gizmo_description/urdf/include/robot_components/caster_wheel.xacro (robot description, xacro)
@@ -7,5 +7,5 @@
     <xacro:property name="caster_wheel_o_rpy" value="0 0 0" />
     <!-- Link caster_wheel -->
-    <link name="caster_wheel">
+    <link name="${tf_prefix}caster_wheel">
         <xacro:sphere_inertia m="${caster_wheel_m}" r="${caster_wheel_r}" o_xyz="${caster_wheel_o_xyz}" o_rpy="${caster_wheel_o_rpy}"/>
         <collision>

File: src/gizmo_description/urdf/include/robot_components/gizmo_mobile_base.xacro (robot description, xacro)
@@ -15,34 +15,34 @@
     <xacro:property name="base_floor1_wheel_right_o_xyz" value="0.03 -0.0691386 0.01986" />
     <!-- Link base_footprint -->
-    <link name="base_footprint"/>
+    <link name="${tf_prefix}base_footprint"/>
     <!-- Joint base_footprint_base_floor1 -->
     <joint name="base_footprint_joint" type="fixed">
         <origin xyz="${base_footprint_base_floor1_o_xyz}" rpy="0 0 0"/>
-        <parent link="base_footprint"/>
-        <child link="base_floor1"/>
+        <parent link="${tf_prefix}base_footprint"/>
+        <child link="${tf_prefix}base_floor1"/>
     </joint>
     <!-- Joint base_floor1_base_floor2 -->
     <joint name="base_floor1_base_floor2_joint" type="fixed">
         <origin xyz="${base_floor1_base_floor2_o_xyz}" rpy="0 0 0"/>
-        <parent link="base_floor1"/>
-        <child link="base_floor2"/>
+        <parent link="${tf_prefix}base_floor1"/>
+        <child link="${tf_prefix}base_floor2"/>
     </joint>
     <!-- Joint base_floor2_base_floor3 -->
     <joint name="base_floor2_base_floor3_joint" type="fixed">
         <origin xyz="${base_floor2_base_floor3_o_xyz}" rpy="0 0 0"/>
-        <parent link="base_floor2"/>
-        <child link="base_floor3"/>
+        <parent link="${tf_prefix}base_floor2"/>
+        <child link="${tf_prefix}base_floor3"/>
     </joint>
     <!-- Joint base_floor1_caster_wheel -->
     <joint name="caster_wheel_joint" type="fixed">
         <origin xyz="${base_floor1_caster_wheel_o_xyz}" rpy="0 0 0"/>
-        <parent link="base_floor1"/>
-        <child link="caster_wheel"/>
+        <parent link="${tf_prefix}base_floor1"/>
+        <child link="${tf_prefix}caster_wheel"/>
     </joint>
     <!-- Joint base_floor1_wheel_left -->
     <joint name="left_wheel_joint" type="continuous">
         <origin xyz="${base_floor1_wheel_left_o_xyz}" rpy="0 0 0"/>
-        <parent link="base_floor1"/>
-        <child link="wheel_left"/>
+        <parent link="${tf_prefix}base_floor1"/>
+        <child link="${tf_prefix}wheel_left"/>
         <axis xyz="0 1 0"/>
         <!-- <limit effort="10" velocity="10"/> -->
@@ -51,6 +51,6 @@
     <joint name="right_wheel_joint" type="continuous">
         <origin xyz="${base_floor1_wheel_right_o_xyz}" rpy="0 0 0"/>
-        <parent link="base_floor1"/>
-        <child link="wheel_right"/>
+        <parent link="${tf_prefix}base_floor1"/>
+        <child link="${tf_prefix}wheel_right"/>
         <axis xyz="0 1 0"/>
         <!-- <limit effort="10" velocity="10"/> -->

File: src/gizmo_description/urdf/include/robot_components/imu.xacro (robot description, xacro)
@@ -9,5 +9,5 @@
     <xacro:property name="imu_o_rpy" value="0 0 0" />
     <!-- Link imu_link -->
-    <link name="imu_link">
+    <link name="${tf_prefix}imu_link">
         <xacro:box_inertia m="${imu_m}" x="${imu_length}" y="${imu_width}" z="${imu_height}" o_xyz="${imu_o_xyz}" o_rpy="${imu_o_rpy}"/>
         <collision>

File: src/gizmo_description/urdf/include/robot_components/lidar.xacro (robot description, xacro)
@@ -7,5 +7,5 @@
     <xacro:property name="lidar_o_rpy" value="0 0 0" />
     <!-- Link lidar_link -->
-    <link name="lidar_link">
+    <link name="${tf_prefix}lidar_link">
         <xacro:cylinder_inertia m="${lidar_m}" r="${lidar_r}" h="${lidar_length}" o_xyz="${lidar_o_xyz}" o_rpy="${lidar_o_rpy}"/>
         <collision>
@@ -26,4 +26,4 @@
         </visual>
     </link>
-    <link name="scan_frame"/>
+    <link name="${tf_prefix}scan_frame"/>
 </robot>

File: src/gizmo_description/urdf/include/robot_components/sensors.xacro (robot description, xacro)
@@ -21,28 +21,28 @@
     <joint name="lidar_link_joint" type="fixed">
         <origin xyz="${base_floor3_lidar_link_o_xyz}" rpy="${base_floor3_lidar_link_o_rpy}"/>
-        <parent link="base_floor3"/>
-        <child link="lidar_link"/>
+        <parent link="${tf_prefix}base_floor3"/>
+        <child link="${tf_prefix}lidar_link"/>
     </joint>
     <joint name="scan_frame_joint" type="fixed">
         <origin xyz="${lidar_scan_frame_o_xyz}" rpy="${lidar_scan_frame_o_rpy}"/>
-        <parent link="lidar_link"/>
-        <child link="scan_frame"/>
+        <parent link="${tf_prefix}lidar_link"/>
+        <child link="${tf_prefix}scan_frame"/>
     </joint>
     <!-- Joint camera_link -->
     <joint name="camera_link_joint" type="fixed">
         <origin xyz="${base_floor3_camera_link_o_xyz}" rpy="${base_floor3_camera_link_o_rpy}"/>
-        <parent link="base_floor3"/>
-        <child link="camera_link"/>
+        <parent link="${tf_prefix}base_floor3"/>
+        <child link="${tf_prefix}camera_link"/>
     </joint>
     <joint name="camera_optical_frame_joint" type="fixed">
         <origin xyz="${camera_optical_frame_o_xyz}" rpy="${camera_optical_frame_o_rpy}"/>
-        <parent link="camera_link"/>
-        <child link="camera_optical_frame"/>
+        <parent link="${tf_prefix}camera_link"/>
+        <child link="${tf_prefix}camera_optical_frame"/>
     </joint>
     <!-- Joint imu_link -->
     <joint name="imu_link_joint" type="fixed">
         <origin xyz="${base_floor1_imu_link_o_xyz}" rpy="${base_floor1_imu_link_o_rpy}"/>
-        <parent link="base_floor1"/>
-        <child link="imu_link"/>
+        <parent link="${tf_prefix}base_floor1"/>
+        <child link="${tf_prefix}imu_link"/>
     </joint>
 </robot>

File: src/gizmo_description/urdf/include/robot_components/wheel_left.xacro (robot description, xacro)
@@ -4,5 +4,5 @@
     <xacro:property name="wheel_left_set_o_xyz" value="0 -0.0025 0" />
     <xacro:property name="wheel_left_set_o_rpy" value="${pi/2} 0 0" />
-    xacro:<xacro:property name="wheel_left_set_h" value="0.0130" />
+    <xacro:property name="wheel_left_set_h" value="0.0130" />
     <xacro:property name="wheel_left_d" value="0.070" />
     <xacro:property name="wheel_left_r" value="${wheel_left_d / 2}" />
@@ -10,5 +10,5 @@
     <xacro:property name="wheel_left_o_rpy" value="0 0 0" />
   <!-- Link wheel_left -->
-  <link name="wheel_left">
+  <link name="${tf_prefix}wheel_left">
     <xacro:cylinder_inertia m="${wheel_left_set_m}" r="${wheel_left_r}" h="${wheel_left_set_h}" o_xyz="${wheel_left_set_o_xyz}" o_rpy="${wheel_left_set_o_rpy}"/>
     <collision>

File: src/gizmo_description/urdf/include/robot_components/wheel_right.xacro (robot description, xacro)
@@ -4,5 +4,5 @@
     <xacro:property name="wheel_right_set_o_xyz" value="0 0.0025 0" />
     <xacro:property name="wheel_right_set_o_rpy" value="${pi/2} 0 0" />
-    xacro:<xacro:property name="wheel_right_set_h" value="0.0130" />
+    <xacro:property name="wheel_right_set_h" value="0.0130" />
     <xacro:property name="wheel_right_d" value="0.070" />
     <xacro:property name="wheel_right_r" value="${wheel_right_d / 2}" />
@@ -10,5 +10,5 @@
     <xacro:property name="wheel_right_o_rpy" value="0 0 0" />
 <!-- Link wheel_right -->
-  <link name="wheel_right">
+  <link name="${tf_prefix}wheel_right">
     <xacro:cylinder_inertia m="${wheel_right_set_m}" r="${wheel_right_r}" h="${wheel_right_set_h}" o_xyz="${wheel_right_set_o_xyz}" o_rpy="${wheel_right_set_o_rpy}"/>
     <collision>

Commit message: fix(gizmo_description): sanitize prefix argument in xacro - Strip leading and trailing slashes from raw prefix input - Ensure tf_prefix never starts with '/' to comply with ROS 2 tf2 rules - Ensure topic_prefix always starts and ends with '/' for sensor topics

File: src/gizmo_description/urdf/gizmo.urdf.xacro (robot description, xacro)
@@ -2,7 +2,11 @@
 <robot name="gizmo" xmlns:xacro="http://www.ros.org/wiki/xacro">
     <xacro:arg name="prefix" default="" />
-    <xacro:property name="_prefix" value="$(arg prefix)" />
-    <xacro:property name="tf_prefix" value="${_prefix if (_prefix == '' or _prefix.endswith('/')) else _prefix + '/'}" />
-    <xacro:property name="topic_prefix" value="${('/' + tf_prefix) if not tf_prefix.startswith('/') else tf_prefix}" />
+    <xacro:property name="_raw_prefix" value="$(arg prefix)" />
+    <!-- Strip all leading and trailing slashes first -->
+    <xacro:property name="_prefix" value="${_raw_prefix.strip('/')}" />
+    <!-- If not empty, add trailing slash for TF; otherwise keep empty -->
+    <xacro:property name="tf_prefix" value="${(_prefix + '/') if _prefix else ''}" />
+    <!-- Always start with '/' for ROS topics -->
+    <xacro:property name="topic_prefix" value="${('/' + _prefix + '/') if _prefix else '/'}" />
     <xacro:include filename="$(find gizmo_description)/urdf/include/robot_components/gizmo_mobile_base.xacro" />
     <xacro:include filename="$(find gizmo_description)/urdf/include/gazebo_components/gizmo_mobile_base.gazebo.xacro" />
